Commit message: adds a complete visual urdf

File: urdf/diff_drive.urdf (robot description, URDF)
Before this commit: robot gz_example_robot, 1 links, 0 joints
Links:
- added link chassis_link
- added link front_wheel; visual sphere radius=0.02
- added link left_wheel; visual cylinder length=0.04 radius=0.08
- added link right_wheel; visual cylinder length=0.04 radius=0.08
- link base_link: geometry visual box size=0.24 0.16 0.12
Joints:
- added joint chassis_joint: type fixed, parent base_link, child chassis_link, origin xyz=0.08 0 0.06 rpy=0 0 0
- added joint front_wheel_joint: type fixed, parent base_link, child front_wheel, origin xyz=0.18 0 -0.06 rpy=0 0 0
- added joint left_wheel_joint: type continuous, parent base_link, child left_wheel, origin xyz=0 0.08 -0.02 rpy=-1.5708 0 0, axis 0 0 1
- added joint right_wheel_joint: type continuous, parent base_link, child right_wheel, origin xyz=0 -0.08 -0.02 rpy=-1.5708 0 0, axis 0 0 1
