Commit message: Full working urdf.xacro with lidar, diffdrive, imu

File: urdf/diff_drive_simulation.urdf.xacro (robot description, xacro)
@@ -11,4 +11,5 @@
 <xacro:property name="base_offset"      value="0.08" />
 <xacro:property name="footprint_z"      value="${chassis_height/2 + sphere_radius}" />
+<xacro:property name="control_config"   value="$(find gz_example_robot_description)/config/diff_drive_control.yaml" />
   <!-- LINKS -->
   <link name="base_footprint"/>
@@ -163,28 +164,144 @@
   </joint>
   <!-- GAZEBO PLUGINS -->
+  <!-- Differential Drive - https://gazebosim.org/api/gazebo/4.5/classignition_1_1gazebo_1_1systems_1_1DiffDrive.html -->
   <gazebo>
     <plugin filename="ignition-gazebo-diff-drive-system" name="ignition::gazebo::systems::DiffDrive">
-      <!-- wheels -->
+      <!-- Wheel Joints -->
       <left_joint>left_wheel_joint</left_joint>
       <right_joint>right_wheel_joint</right_joint>
-      <!-- kinematics -->
-      <wheel_separation>0.16</wheel_separation>
-      <wheel_diameter>0.16</wheel_diameter>
-      <!-- limits -->
-      <max_wheel_torque>20</max_wheel_torque>
-      <max_wheel_acceleration>1.0</max_wheel_acceleration>
-      <!-- output -->
-      <publish_odom>true</publish_odom>
-      <publish_wheel_tf>true</publish_wheel_tf>
-      <publish_odom_tf>false</publish_odom_tf>
-      <odometry_frame>odom</odometry_frame>
-      <robot_base_frame>base_link</robot_base_frame>
-      <topic>/model/gz_example_robot/cmd_vel</topic>
-      <odom_topic>/model/gz_example_robot/odometry</odom_topic>
+      <!-- Kinematics -->
+      <wheel_separation>${wheel_separation}</wheel_separation>
+      <wheel_radius>${wheel_radius}</wheel_radius>
+      <odom_publish_frequency>50</odom_publish_frequency>
+      <!-- TF Frames -->
+      <frame_id>/odom</frame_id>
+      <child_frame_id>/base_footprint</child_frame_id>
+      <!-- topics -->
+      <!-- <topic>/model/gz_example_robot/cmd_vel</topic> THIS IS DEFAULT -->
+      <!-- <odom_topic>/model/gz_example_robot/odometry</odom_topic> THIS IS DEFAULT-->
+      <!-- <tf_topic>/model/gz_example_robot/tf</tf_topic> THIS IS DEFAULT -->
+      <!-- <tf_topic></tf_topic> Leave blank if you plan to use a filter + imu (e.g. EKF) -->
     </plugin>
   </gazebo>
-  <gazebo reference="front_wheel_wheel">
+  <gazebo>
+      <plugin filename="ignition-gazebo-joint-state-publisher-system" name="ignition::gazebo::systems::JointStatePublisher">
+        <update_rate>50</update_rate>
+        <joint_name>left_wheel_joint</joint_name>
+        <joint_name>right_wheel_joint</joint_name>
+      </plugin>
+  </gazebo>
+  <gazebo reference="front_wheel">
     <mu1 value="0.001"/>
     <mu2 value="0.001"/>
   </gazebo>
+  <gazebo reference="right_wheel">
+    <mu1 value="0.8"/>
+    <mu2 value="0.8"/>
+  </gazebo>
+  <gazebo reference="left_wheel">
+    <mu1 value="0.8"/>
+    <mu2 value="0.8"/>
+  </gazebo>
+  <gazebo reference="lidar_link">
+    <sensor type="gpu_lidar" name="generic_lidar_sensor">
+      <topic>/model/gz_example_robot/scan</topic>
+      <frame_id>lidar_link</frame_id>
+      <ignition_frame_id>lidar_link</ignition_frame_id>
+      <update_rate>10.0</update_rate>
+      <ray>
+        <scan>
+          <horizontal>
+            <samples>512</samples>
+            <resolution>1</resolution>
+            <min_angle>-${pi*0.75}</min_angle>
+            <max_angle>${pi*0.75}</max_angle>
+          </horizontal>
+        </scan>
+        <range>
+          <min>0.10</min>
+          <max>10.0</max>
+          <resolution>0.03</resolution>
+        </range>
+        <noise>
+          <type>gaussian</type>
+          <mean>0.0</mean>
+          <stddev>0.001</stddev>
+        </noise>
+      </ray>
+      <always_on>1</always_on>
+      <visualize>false</visualize>
+    </sensor>
+  </gazebo>
+  <gazebo>
+    <plugin filename="libignition-gazebo-sensors-system.so" name="ignition::gazebo::systems::Sensors">
+      <render_engine>ogre2</render_engine>
+    </plugin>
+  </gazebo>
+  <gazebo reference="imu_link">
+    <sensor name="imu_sensor" type="imu">
+      <topic>/model/gz_example_robot/imu</topic>
+      <frame_id>imu_link</frame_id>
+      <ignition_frame_id>imu_link</ignition_frame_id>
+      <plugin filename="libignition-gazebo-imu-system.so" name="ignition::gazebo::systems::Imu">
+        <initial_orientation_as_reference>false</initial_orientation_as_reference>
+      </plugin>
+      <always_on>true</always_on>
+      <update_rate>100</update_rate>
+      <visualize>true</visualize>
+     <imu>
+     	<angular_velocity>
+     	  <x>
+     	    <noise type="gaussian">
+              <mean>0.0</mean>
+              <stddev>2e-4</stddev>
+              <bias_mean>0.0000075</bias_mean>
+              <bias_stddev>0.0000008</bias_stddev>
+            </noise>
+          </x>
+          <y>
+            <noise type="gaussian">
+              <mean>0.0</mean>
+              <stddev>2e-4</stddev>
+              <bias_mean>0.0000075</bias_mean>
+              <bias_stddev>0.0000008</bias_stddev>
+            </noise>
+          </y>
+          <z>
+            <noise type="gaussian">
+              <mean>0.0</mean>
+              <stddev>2e-4</stddev>
+              <bias_mean>0.0000075</bias_mean>
+              <bias_stddev>0.0000008</bias_stddev>
+            </noise>
+          </z>
+        </angular_velocity>
+        <linear_acceleration>
+          <x>
+            <noise type="gaussian">
+              <mean>0.0</mean>
+              <stddev>1.7e-2</stddev>
+              <bias_mean>0.1</bias_mean>
+              <bias_stddev>0.001</bias_stddev>
+            </noise>
+          </x>
+          <y>
+            <noise type="gaussian">
+              <mean>0.0</mean>
+              <stddev>1.7e-2</stddev>
+              <bias_mean>0.1</bias_mean>
+              <bias_stddev>0.001</bias_stddev>
+            </noise>
+          </y>
+          <z>
+            <noise type="gaussian">
+              <mean>0.0</mean>
+              <stddev>1.7e-2</stddev>
+              <bias_mean>0.1</bias_mean>
+              <bias_stddev>0.001</bias_stddev>
+            </noise>
+          </z>
+        </linear_acceleration>
+      </imu>
+    </sensor>
+  </gazebo>
 </robot>
